Commit message: update GGC_TestModel_rx78_20170112.urdf and gundam_rx78_control.yaml with latest ggc_dae_to_urdf.py

File: gundam_rx78_description/urdf/GGC_TestModel_rx78_20170112.urdf (robot description, URDF)
Before this commit: robot GGC_TestModel_rx78_20170112, 182 links, 181 joints
Links:
- removed link world
- link base_link: mass 0.8 -> None; geometry 
- link rx78_Null_005_link: mass 0.8 -> None; geometry 
- link rx78_Null_006_link: mass 0.8 -> None; geometry 
- link rx78_Null_007_link: mass 0.8 -> None; geometry 
- link rx78_Null_008_link: mass 0.8 -> None; geometry 
- link rx78_Null_009_link: mass 0.8 -> None; geometry 
- link rx78_Null_010_link: mass 0.8 -> None; geometry 
- link rx78_Null_011_link: mass 0.8 -> None; geometry 
- link rx78_Null_012_link: mass 0.8 -> None; geometry 
- link rx78_Null_013_link: mass 0.8 -> None; geometry 
- link rx78_Null_035_link: mass 0.8 -> 256.0; geometry collision box size=1.0 0.8 0.8
- link rx78_Null_042_link: mass 0.8 -> None; geometry 
- link rx78_Null_043_link: mass 0.8 -> None; geometry 
- link rx78_Null_044_link: mass 0.8 -> None; geometry 
- link rx78_Null_045_link: mass 0.8 -> None; geometry 
- link rx78_Null_048_link: mass 0.8 -> None; geometry 
- link rx78_Null_065_link: mass 0.8 -> None; geometry 
- link rx78_Null_081_link: mass 0.8 -> None; geometry 
- link rx78_Null_082_link: mass 0.8 -> None; geometry 
- link rx78_Null_085_link: mass 0.8 -> 256.0; geometry collision box size=1.0 0.8 0.8
- link rx78_Null_092_link: mass 0.8 -> None; geometry 
- link rx78_Null_093_link: mass 0.8 -> None; geometry 
- link rx78_Null_094_link: mass 0.8 -> None; geometry 
- link rx78_Null_095_link: mass 0.8 -> None; geometry 
- link rx78_object_010_link: mass 1.95924236277 -> 50
- link rx78_object_012_link: mass 1.59685738091 -> 50
- link rx78_object_013_link: mass 2.36426706662 -> 50
- link rx78_object_014_link: mass 1.42045159698 -> 50
- link rx78_object_015_link: mass 1.59685874833 -> 50
- link rx78_object_016_link: mass 2.36427062486 -> 50
- link rx78_object_017_link: mass 1.42045355099 -> 50
- link rx78_object_018_link: mass 1.59685613286 -> 50
- link rx78_object_019_link: mass 2.36427035847 -> 50
- link rx78_object_020_link: mass 1.42045397774 -> 50
- link rx78_object_023_link: mass 570.711450018 -> 856.067175028
- link rx78_object_032_link: mass 330.049913295 -> 1650.24956648
- link rx78_object_041_link: mass 570.711053625 -> 856.066580437
- link rx78_object_047_link: mass 12.7891829509 -> 50
- link rx78_object_049_link: mass 1.59685469138 -> 50
- link rx78_object_050_link: mass 2.36426949429 -> 50
- link rx78_object_051_link: mass 3.39819719842 -> 50
- link rx78_object_052_link: mass 2.36428302837 -> 50
- link rx78_object_053_link: mass 1.42045209647 -> 50
- link rx78_object_054_link: mass 1.59685842145 -> 50
- link rx78_object_055_link: mass 2.36429121821 -> 50
- link rx78_object_056_link: mass 1.42044976922 -> 50
- link rx78_object_057_link: mass 1.59685707602 -> 50
- link rx78_object_058_link: mass 2.36425622333 -> 50
- link rx78_object_059_link: mass 3.39818789121 -> 50
- link rx78_object_061_link: mass 12.789270605 -> 50
- link rx78_object_062_link: mass 220.380043855 -> 330.570065783
- link rx78_object_065_link: mass 1.5968575337 -> 50
- link rx78_object_066_link: mass 2.36427951181 -> 50
- link rx78_object_067_link: mass 1.42044821773 -> 50
- link rx78_object_068_link: mass 1.59685629149 -> 50
- link rx78_object_069_link: mass 2.36428387843 -> 50
- link rx78_object_070_link: mass 1.4204498081 -> 50
- link rx78_object_071_link: mass 1.59685684283 -> 50
- link rx78_object_072_link: mass 1.59685806327 -> 50
- link rx78_object_073_link: mass 2.3642746058 -> 50
- link rx78_object_074_link: mass 1.42045361411 -> 50
- link rx78_object_076_link: mass 221.302180541 -> 331.953270811
- link rx78_object_089_link: mass 330.052784029 -> 1650.26392015
Joints:
- removed joint rx78_Null_056_joint
- removed joint rx78_Null_062_joint
- removed joint world_to_base
- added joint rx78_Null_021_joint: type revolute, parent rx78_Null_055_link, child rx78_Null_021_link, origin xyz=0.068401 -0.105633 -0.907139 rpy=0.0 -0.0 0.0, axis 0 -1 0, limit lower=-1.57079632679 upper=1.57079632679 effort=1000000000 velocity=1000000, mimic joint=rarm_gripper
- added joint rx78_Null_059_joint: type revolute, parent rx78_Null_069_link, child rx78_Null_059_link, origin xyz=-0.0683779 -0.31073 -0.853204 rpy=-9.99999997475e-07 -0.0 0.0, axis 0 1 0, limit lower=-1.57079632679 upper=1.57079632679 effort=1000000000 velocity=1000000, mimic joint=larm_gripper
- joint head_neck_p: limit lower=-0.628318530718 upper=1.57079632679 effort=10000000 velocity=1000000 -> lower=-0.628318530718 upper=1.57079632679 effort=1000000000 velocity=1000000
- joint head_neck_y: limit lower=-1.57079632679 upper=1.57079632679 effort=10000000 velocity=1000000 -> lower=-1.57079632679 upper=1.57079632679 effort=1000000000 velocity=1000000
- joint larm_elbow_p: limit lower=-1.0471975512 upper=0.1308996939 effort=10000000 velocity=1000000 -> lower=-1.0471975512 upper=0.1308996939 effort=1000000000 velocity=1000000
- joint larm_gripper: child rx78_Null_059_link -> rx78_Null_062_link; limit lower=-0.1308996939 upper=1.57079632679 effort=10000000 velocity=1000000 -> lower=-0.1308996939 upper=1.57079632679 effort=1000000000 velocity=1000000; origin xyz=-0.0683779 -0.31073 -0.853204 rpy=-9.99999997475e-07 -0.0 0.0 -> xyz=-0.265212 -0.284142 -0.0825119 rpy=0.0 1.99999999495e-06 0.0
- joint larm_shoulder_p: limit lower=-1.57079632679 upper=1.57079632679 effort=10000000 velocity=1000000 -> lower=-1.57079632679 upper=1.57079632679 effort=1000000000 velocity=1000000
- joint larm_shoulder_r: limit lower=-0.523598775598 upper=1.57079632679 effort=10000000 velocity=1000000 -> lower=-0.523598775598 upper=1.57079632679 effort=1000000000 velocity=1000000
- joint larm_shoulder_y: limit lower=-1.57079632679 upper=1.57079632679 effort=10000000 velocity=1000000 -> lower=-1.57079632679 upper=1.57079632679 effort=1000000000 velocity=1000000
- joint larm_wrist_r: limit lower=-1.57079632679 upper=1.57079632679 effort=10000000 velocity=1000000 -> lower=-1.57079632679 upper=1.57079632679 effort=1000000000 velocity=1000000
- joint larm_wrist_y: limit lower=-1.57079632679 upper=1.57079632679 effort=10000000 velocity=1000000 -> lower=-1.57079632679 upper=1.57079632679 effort=1000000000 velocity=1000000
- joint lleg_ankle_p: limit lower=-0.785398163397 upper=0.785398163397 effort=10000000 velocity=1000000 -> lower=-0.785398163397 upper=0.785398163397 effort=1000000000 velocity=1000000
- joint lleg_ankle_r: limit lower=-0.261799387799 upper=0.261799387799 effort=10000000 velocity=1000000 -> lower=-0.261799387799 upper=0.261799387799 effort=1000000000 velocity=1000000
- joint lleg_crotch_p: limit lower=-0.785398163397 upper=0.785398163397 effort=10000000 velocity=1000000 -> lower=-0.785398163397 upper=0.785398163397 effort=1000000000 velocity=1000000
- joint lleg_crotch_r: limit lower=-0.261799387799 upper=0.785398163397 effort=10000000 velocity=1000000 -> lower=-0.261799387799 upper=0.785398163397 effort=1000000000 velocity=1000000
- joint lleg_crotch_y: limit lower=-1.57079632679 upper=1.57079632679 effort=10000000 velocity=1000000 -> lower=-1.57079632679 upper=1.57079632679 effort=1000000000 velocity=1000000
- joint lleg_knee_p: limit lower=-0.1308996939 upper=1.0471975512 effort=10000000 velocity=1000000 -> lower=-0.1308996939 upper=1.0471975512 effort=1000000000 velocity=1000000
- joint rarm_elbow_p: limit lower=-1.0471975512 upper=0.1308996939 effort=10000000 velocity=1000000 -> lower=-1.0471975512 upper=0.1308996939 effort=1000000000 velocity=1000000
- joint rarm_gripper: child rx78_Null_021_link -> rx78_Null_056_link; limit lower=-0.1308996939 upper=1.57079632679 effort=10000000 velocity=1000000 -> lower=-0.1308996939 upper=1.57079632679 effort=1000000000 velocity=1000000; origin xyz=0.068401 -0.105633 -0.907139 rpy=0.0 -0.0 0.0 -> xyz=0.2652 -0.284142 -0.112511 rpy=0.0 -0.0 0.0
- joint rarm_shoulder_p: limit lower=-1.57079632679 upper=1.57079632679 effort=10000000 velocity=1000000 -> lower=-1.57079632679 upper=1.57079632679 effort=1000000000 velocity=1000000
- joint rarm_shoulder_r: limit lower=-1.57079632679 upper=0.523598775598 effort=10000000 velocity=1000000 -> lower=-1.57079632679 upper=0.523598775598 effort=1000000000 velocity=1000000
- joint rarm_shoulder_y: limit lower=-1.57079632679 upper=1.57079632679 effort=10000000 velocity=1000000 -> lower=-1.57079632679 upper=1.57079632679 effort=1000000000 velocity=1000000
- joint rarm_wrist_r: limit lower=-1.57079632679 upper=1.57079632679 effort=10000000 velocity=1000000 -> lower=-1.57079632679 upper=1.57079632679 effort=1000000000 velocity=1000000
- joint rarm_wrist_y: limit lower=-1.57079632679 upper=1.57079632679 effort=10000000 velocity=1000000 -> lower=-1.57079632679 upper=1.57079632679 effort=1000000000 velocity=1000000
- joint rleg_ankle_p: limit lower=-0.785398163397 upper=0.785398163397 effort=10000000 velocity=1000000 -> lower=-0.785398163397 upper=0.785398163397 effort=1000000000 velocity=1000000
- joint rleg_ankle_r: limit lower=-0.261799387799 upper=0.261799387799 effort=10000000 velocity=1000000 -> lower=-0.261799387799 upper=0.261799387799 effort=1000000000 velocity=1000000
- joint rleg_crotch_p: limit lower=-0.785398163397 upper=0.785398163397 effort=10000000 velocity=1000000 -> lower=-0.785398163397 upper=0.785398163397 effort=1000000000 velocity=1000000
- joint rleg_crotch_r: limit lower=-0.785398163397 upper=0.261799387799 effort=10000000 velocity=1000000 -> lower=-0.785398163397 upper=0.261799387799 effort=1000000000 velocity=1000000
- joint rleg_crotch_y: limit lower=-1.57079632679 upper=1.57079632679 effort=10000000 velocity=1000000 -> lower=-1.57079632679 upper=1.57079632679 effort=1000000000 velocity=1000000
- joint rleg_knee_p: limit lower=-0.1308996939 upper=1.0471975512 effort=10000000 velocity=1000000 -> lower=-0.1308996939 upper=1.0471975512 effort=1000000000 velocity=1000000
- joint rx78_Null_016_joint: limit lower=-1.57079632679 upper=1.57079632679 effort=10000000 velocity=1000000 -> lower=-1.57079632679 upper=1.57079632679 effort=1000000000 velocity=1000000
- joint rx78_Null_022_joint: limit lower=-1.57079632679 upper=1.57079632679 effort=10000000 velocity=1000000 -> lower=-1.57079632679 upper=1.57079632679 effort=1000000000 velocity=1000000
- joint rx78_Null_023_joint: limit lower=-1.57079632679 upper=1.57079632679 effort=10000000 velocity=1000000 -> lower=-1.57079632679 upper=1.57079632679 effort=1000000000 velocity=1000000
- joint rx78_Null_024_joint: limit lower=-1.57079632679 upper=1.57079632679 effort=10000000 velocity=1000000 -> lower=-1.57079632679 upper=1.57079632679 effort=1000000000 velocity=1000000
- joint rx78_Null_025_joint: limit lower=-1.57079632679 upper=1.57079632679 effort=10000000 velocity=1000000 -> lower=-1.57079632679 upper=1.57079632679 effort=1000000000 velocity=1000000
- joint rx78_Null_026_joint: limit lower=-1.57079632679 upper=1.57079632679 effort=10000000 velocity=1000000 -> lower=-1.57079632679 upper=1.57079632679 effort=1000000000 velocity=1000000
- joint rx78_Null_027_joint: limit lower=-1.57079632679 upper=1.57079632679 effort=10000000 velocity=1000000 -> lower=-1.57079632679 upper=1.57079632679 effort=1000000000 velocity=1000000
- joint rx78_Null_028_joint: limit lower=-1.57079632679 upper=1.57079632679 effort=10000000 velocity=1000000 -> lower=-1.57079632679 upper=1.57079632679 effort=1000000000 velocity=1000000
- joint rx78_Null_029_joint: limit lower=-1.57079632679 upper=1.57079632679 effort=10000000 velocity=1000000 -> lower=-1.57079632679 upper=1.57079632679 effort=1000000000 velocity=1000000
- joint rx78_Null_030_joint: limit lower=-1.57079632679 upper=1.57079632679 effort=10000000 velocity=1000000 -> lower=-1.57079632679 upper=1.57079632679 effort=1000000000 velocity=1000000
- joint rx78_Null_031_joint: limit lower=-1.57079632679 upper=1.57079632679 effort=10000000 velocity=1000000 -> lower=-1.57079632679 upper=1.57079632679 effort=1000000000 velocity=1000000
- joint rx78_Null_032_joint: limit lower=-1.57079632679 upper=1.57079632679 effort=10000000 velocity=1000000 -> lower=-1.57079632679 upper=1.57079632679 effort=1000000000 velocity=1000000; mimic joint=rleg_crotch_r multiplier=-0.5 -> joint=rleg_crotch_r multiplier=-0.6
- joint rx78_Null_033_joint: limit lower=-1.57079632679 upper=1.57079632679 effort=10000000 velocity=1000000 -> lower=-1.57079632679 upper=1.57079632679 effort=1000000000 velocity=1000000
- joint rx78_Null_034_joint: limit lower=-1.57079632679 upper=1.57079632679 effort=10000000 velocity=1000000 -> lower=-1.57079632679 upper=1.57079632679 effort=1000000000 velocity=1000000
- joint rx78_Null_038_joint: limit lower=-1.57079632679 upper=1.57079632679 effort=10000000 velocity=1000000 -> lower=-1.57079632679 upper=1.57079632679 effort=1000000000 velocity=1000000
- joint rx78_Null_040_joint: limit lower=-1.57079632679 upper=1.57079632679 effort=10000000 velocity=1000000 -> lower=-1.57079632679 upper=1.57079632679 effort=1000000000 velocity=1000000
- joint rx78_Null_046_joint: limit lower=-1.57079632679 upper=1.57079632679 effort=10000000 velocity=1000000 -> lower=-1.57079632679 upper=1.57079632679 effort=1000000000 velocity=1000000
- joint rx78_Null_047_joint: limit lower=-1.57079632679 upper=1.57079632679 effort=10000000 velocity=1000000 -> lower=-1.57079632679 upper=1.57079632679 effort=1000000000 velocity=1000000; mimic joint=lleg_crotch_r multiplier=-0.5 -> joint=lleg_crotch_r multiplier=-0.6
- joint rx78_Null_053_joint: limit lower=-1.57079632679 upper=1.57079632679 effort=10000000 velocity=1000000 -> lower=-1.57079632679 upper=1.57079632679 effort=1000000000 velocity=1000000
- joint rx78_Null_057_joint: limit lower=-1.57079632679 upper=1.57079632679 effort=10000000 velocity=1000000 -> lower=-1.57079632679 upper=1.57079632679 effort=1000000000 velocity=1000000
- joint rx78_Null_058_joint: limit lower=-1.57079632679 upper=1.57079632679 effort=10000000 velocity=1000000 -> lower=-1.57079632679 upper=1.57079632679 effort=1000000000 velocity=1000000
- joint rx78_Null_060_joint: limit lower=-1.57079632679 upper=1.57079632679 effort=10000000 velocity=1000000 -> lower=-1.57079632679 upper=1.57079632679 effort=1000000000 velocity=1000000
- joint rx78_Null_061_joint: limit lower=-1.57079632679 upper=1.57079632679 effort=10000000 velocity=1000000 -> lower=-1.57079632679 upper=1.57079632679 effort=1000000000 velocity=1000000
- joint rx78_Null_063_joint: limit lower=-1.57079632679 upper=1.57079632679 effort=10000000 velocity=1000000 -> lower=-1.57079632679 upper=1.57079632679 effort=1000000000 velocity=1000000
- joint rx78_Null_064_joint: limit lower=-1.57079632679 upper=1.57079632679 effort=10000000 velocity=1000000 -> lower=-1.57079632679 upper=1.57079632679 effort=1000000000 velocity=1000000
- joint rx78_Null_066_joint: limit lower=-1.57079632679 upper=1.57079632679 effort=10000000 velocity=1000000 -> lower=-1.57079632679 upper=1.57079632679 effort=1000000000 velocity=1000000
- joint rx78_Null_068_joint: limit lower=-1.57079632679 upper=1.57079632679 effort=10000000 velocity=1000000 -> lower=-1.57079632679 upper=1.57079632679 effort=1000000000 velocity=1000000
- joint rx78_Null_070_joint: limit lower=-1.57079632679 upper=1.57079632679 effort=10000000 velocity=1000000 -> lower=-1.57079632679 upper=1.57079632679 effort=1000000000 velocity=1000000
- joint rx78_Null_071_joint: limit lower=-1.57079632679 upper=1.57079632679 effort=10000000 velocity=1000000 -> lower=-1.57079632679 upper=1.57079632679 effort=1000000000 velocity=1000000
- joint rx78_Null_072_joint: limit lower=-1.57079632679 upper=1.57079632679 effort=10000000 velocity=1000000 -> lower=-1.57079632679 upper=1.57079632679 effort=1000000000 velocity=1000000
- joint rx78_Null_073_joint: limit lower=-1.57079632679 upper=1.57079632679 effort=10000000 velocity=1000000 -> lower=-1.57079632679 upper=1.57079632679 effort=1000000000 velocity=1000000
- joint rx78_Null_074_joint: limit lower=-1.57079632679 upper=1.57079632679 effort=10000000 velocity=1000000 -> lower=-1.57079632679 upper=1.57079632679 effort=1000000000 velocity=1000000
- joint rx78_Null_075_joint: limit lower=-1.57079632679 upper=1.57079632679 effort=10000000 velocity=1000000 -> lower=-1.57079632679 upper=1.57079632679 effort=1000000000 velocity=1000000
- joint rx78_Null_076_joint: limit lower=-1.57079632679 upper=1.57079632679 effort=10000000 velocity=1000000 -> lower=-1.57079632679 upper=1.57079632679 effort=1000000000 velocity=1000000
- joint rx78_Null_077_joint: limit lower=-1.57079632679 upper=1.57079632679 effort=10000000 velocity=1000000 -> lower=-1.57079632679 upper=1.57079632679 effort=1000000000 velocity=1000000
- joint rx78_Null_078_joint: limit lower=-1.57079632679 upper=1.57079632679 effort=10000000 velocity=1000000 -> lower=-1.57079632679 upper=1.57079632679 effort=1000000000 velocity=1000000
- joint rx78_Null_079_joint: limit lower=-1.57079632679 upper=1.57079632679 effort=10000000 velocity=1000000 -> lower=-1.57079632679 upper=1.57079632679 effort=1000000000 velocity=1000000
- joint rx78_Null_080_joint: limit lower=-1.57079632679 upper=1.57079632679 effort=10000000 velocity=1000000 -> lower=-1.57079632679 upper=1.57079632679 effort=1000000000 velocity=1000000
- joint rx78_Null_084_joint: limit lower=-1.57079632679 upper=1.57079632679 effort=10000000 velocity=1000000 -> lower=-1.57079632679 upper=1.57079632679 effort=1000000000 velocity=1000000
- joint rx78_Null_088_joint: limit lower=-1.57079632679 upper=1.57079632679 effort=10000000 velocity=1000000 -> lower=-1.57079632679 upper=1.57079632679 effort=1000000000 velocity=1000000
- joint rx78_Null_090_joint: limit lower=-1.57079632679 upper=1.57079632679 effort=10000000 velocity=1000000 -> lower=-1.57079632679 upper=1.57079632679 effort=1000000000 velocity=1000000
- joint torso_waist_p: limit lower=-0.261799387799 upper=0.261799387799 effort=10000000 velocity=1000000 -> lower=-0.785398163397 upper=0.785398163397 effort=1000000000 velocity=1000000
- joint torso_waist_y: limit lower=-0.261799387799 upper=0.261799387799 effort=10000000 velocity=1000000 -> lower=-0.261799387799 upper=0.261799387799 effort=1000000000 velocity=1000000

Commit message: update GGC_TestModel_rx78_20170112.urdf and gundam_rx78_control.yaml with latest ggc_dae_to_urdf.py

File: gundam_rx78_description/urdf/GGC_TestModel_rx78_20170112.urdf (robot description, URDF)
Before this commit: robot GGC_TestModel_rx78_20170112, 181 links, 180 joints
Links:
- link rx78_Null_040_link: mass 0.8 -> None; geometry 
- link rx78_Null_090_link: mass 0.8 -> None; geometry 
- link rx78_object_032_link: mass 1650.24956648 -> 330.049913295
- link rx78_object_089_link: mass 1650.26392015 -> 330.052784029
Joints:
- joint rx78_Null_040_joint: axis -1 0 0 -> (none); limit lower=-1.57079632679 upper=1.57079632679 effort=1000000000 velocity=1000000 -> (none); mimic joint=lleg_ankle_r -> (none); origin xyz=1.9e-06 -6e-07 -0.716289 rpy=0.0 -0.0 1.57079632679 -> xyz=1.44559 0 0 rpy=0 0 0; parent rx78_Null_039_link -> rx78_Null_041_link; type revolute -> fixed
- joint rx78_Null_090_joint: axis -1 0 0 -> (none); limit lower=-1.57079632679 upper=1.57079632679 effort=1000000000 velocity=1000000 -> (none); mimic joint=rleg_ankle_r -> (none); origin xyz=2.99e-05 -5e-07 -0.716289 rpy=3.0000001061e-06 -0.0 1.5707763268 -> xyz=1.44559 0 0 rpy=0 0 0; parent rx78_Null_089_link -> rx78_Null_091_link; type revolute -> fixed
